Commit message: Update multirotor_base.xacro

File: ardupilot_sitl_gazebo_plugin/urdf/multirotor_base.xacro (robot description, xacro)
@@ -47,5 +47,5 @@
       </inertial>
       <visual>
-        <origin xyz="0 0 0" rpy="0 0 0" />
+        <origin xyz="-0.180 -0.180 -0.165" rpy="0 0 0" />
         <geometry>
           <mesh filename="package://ardupilot_sitl_gazebo_plugin/meshes/meshes_drones/${mesh_file}"
